File: HW/MOTOR_TERMINAL_BREAKOUT_25mm.kicad_sch (KiCad schematic)
At the start: 11 parts

Commit message: Update Design for Next MFG Run
Parts:
- removed C1: C_0603, C_Capacitor:C_0603, symbol C_Capacitor:C_0603
- removed H1, H2: MountingHole_Pad, MountingHole:MountingHole_3.2mm_M3_ISO7380_Pad_TopBottom, symbol Mechanical:MountingHole_Pad
- removed H10, H3, H4, H5, H6, H7, H8, H9: MountingHole_Pad, MountingHole:MountingHole_3mm_Pad_TopBottom, symbol Mechanical:MountingHole_Pad
- added C2: 10nF 50V, C_Capacitor:C_0603, symbol C_Capacitor:C_0603
- added M1, M2, M3, M4, M5, M6, M7, M8: 22 Motor Terminal Lead, MOTOR_TERMINAL_BREAKOUT:22 Motor Terminal Lead, symbol MOTOR_TERMINAL_BREAKOUT:22 Motor Terminal Lead
- added N1, N2: Finger_4x5_M1, N_NonPart:Finger_4x5_M1, symbol N_NonPart:Finger_4x5_M1
Connections:
- net +BATT: now also C2.1, M1.1, M2.1, M3.1, M4.1, N1.1
- net GND: now also C2.2, M5.1, M6.1, M7.1, M8.1, N2.1
Other:
- title: N20 FACEPLATE -> MOTOR TERMINAL BREAKOUT 25mm
